Commit message: add forward kinematics

File: quadruped_robot/robot.urdf (robot description, URDF)
Before this commit: robot urdf_door, 13 links, 12 joints
Links:
- added link BL_foot4
- added link BR_foot4
- added link FL_foot4
- added link FR_foot4
Joints:
- added joint BL_joint4: type fixed, parent BL_foot3, child BL_foot4, origin xyz=0 0 -0.2 rpy=0 0 0, axis 0 0 1
- added joint BR_joint4: type fixed, parent BR_foot3, child BR_foot4, origin xyz=0 0 -0.2 rpy=0 0 0, axis 0 0 1
- added joint FL_joint4: type fixed, parent FL_foot3, child FL_foot4, origin xyz=0 0 -0.2 rpy=0 0 0, axis 0 0 1
- added joint FR_joint4: type fixed, parent FR_foot3, child FR_foot4, origin xyz=0 0 -0.2 rpy=0 0 0, axis 0 0 1
